File: Hardware/Kicad/christmas_tree.kicad_pcb (KiCad board)
At the start: 2 copper layers, 88.7 x 98 mm, 61 parts, among them J1 USB_A, J2 Conn_01x06, J3 Touch, SW1 SW_SPDT_shield, U1 TL431LP, U2 TL431LP, U3 ATtiny45-20SU, U4 TTP223

Commit message: added prog
Other:
- board text added: "+"
Changed lines of the file:
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@@
   (general
     (thickness 1.6)
-    (drawings 67)
+    (drawings 79)
     (tracks 421)
     (zones 0)
@@
     )
   )
+  (gr_text + (at 123.4 149.6) (layer Dwgs.User)
+    (effects (font (size 1 1) (thickness 0.15)))
+  )
+  (gr_text + (at 124.4 134.4) (layer Dwgs.User)
+    (effects (font (size 1 1) (thickness 0.15)))
+  )
+  (gr_text + (at 124.6 111.2) (layer Dwgs.User)
+    (effects (font (size 1 1) (thickness 0.15)))
+  )
+  (gr_text + (at 112 121.8) (layer Dwgs.User)
+    (effects (font (size 1 1) (thickness 0.15)))
+  )
+  (gr_text + (at 103.8 104.2) (layer Dwgs.User)
+    (effects (font (size 1 1) (thickness 0.15)))
+  )
+  (gr_text + (at 106.8 87.6) (layer Dwgs.User)
+    (effects (font (size 1 1) (thickness 0.15)))
+  )
+  (gr_text + (at 88.6 85) (layer Dwgs.User)
+    (effects (font (size 1 1) (thickness 0.15)))
+  )
+  (gr_text + (at 128.6 163.8) (layer Dwgs.User)
+    (effects (font (size 1 1) (thickness 0.15)))
+  )
+  (gr_text + (at 75.6 100.8) (layer Dwgs.User)
+    (effects (font (size 1 1) (thickness 0.15)))
+  )
+  (gr_text + (at 83 119.4) (layer Dwgs.User)
+    (effects (font (size 1 1) (thickness 0.15)))
+  )
+  (gr_text + (at 71 130.4) (layer Dwgs.User)
+    (effects (font (size 1 1) (thickness 0.15)))
+  )
+  (gr_text + (at 91.2 139.4) (layer Dwgs.User)
+    (effects (font (size 1 1) (thickness 0.15)))
+  )
   (gr_line (start 117.292509 151.733371) (end 96 126.5) (layer Edge.Cuts) (width 0.05))
